File: Hardware/MotorControlBoard/motorcontrol.sch (EAGLE design)
At the start: 27 parts, among them U1 ATMEGA328P-AU

Commit message: changes in eagle file
Parts:
- 1UF: value CAP-US1206FAB -> 1uF
- C1, C2: value CAP-US1206FAB -> .1uF
- C3: value CAP-US1206FAB -> 10uF
- R10, R11, R12, R13, R14, R15, R16, R2, R3, R4, R5, R6, R7, R8, R9: value (none) -> 0
Changed lines of the file:
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@@
 <part name="U$2" library="fab" deviceset="RESONATOR" device=""/>
 <part name="AVR-ISP" library="fab" deviceset="AVRISP" device="SMD" value=""/>
-<part name="1UF" library="fab" deviceset="CAP-US" device="1206FAB"/>
-<part name="C2" library="fab" deviceset="CAP-US" device="1206FAB"/>
-<part name="C3" library="fab" deviceset="CAP-US" device="1206FAB"/>
+<part name="1UF" library="fab" deviceset="CAP-US" device="1206FAB" value="1uF"/>
+<part name="C2" library="fab" deviceset="CAP-US" device="1206FAB" value=".1uF"/>
+<part name="C3" library="fab" deviceset="CAP-US" device="1206FAB" value="10uF"/>
 <part name="R1" library="fab" deviceset="RES-US" device="1206FAB" value="10K"/>
 <part name="U$3" library="BillPorter" deviceset="AD5290" device=""/>
 <part name="U$4" library="fab" deviceset="PINHD-2X2-SMD" device=""/>
 <part name="0OHM" library="fab" deviceset="RES-US" device="1206FAB"/>
-<part name="R2" library="fab" deviceset="RES-US" device="1206FAB"/>
-<part name="R3" library="fab" deviceset="RES-US" device="1206FAB"/>
-<part name="R4" library="fab" deviceset="RES-US" device="1206FAB"/>
-<part name="R10" library="fab" deviceset="RES-US" device="1206FAB"/>
-<part name="R11" library="fab" deviceset="RES-US" device="1206FAB"/>
-<part name="R12" library="fab" deviceset="RES-US" device="1206"/>
-<part name="R13" library="fab" deviceset="RES-US" device="1206"/>
-<part name="R15" library="fab" deviceset="RES-US" device="1206FAB"/>
-<part name="R5" library="fab" deviceset="RES-US" device="1206FAB"/>
-<part name="R6" library="fab" deviceset="RES-US" device="1206"/>
-<part name="R7" library="fab" deviceset="RES-US" device="1206"/>
-<part name="R8" library="fab" deviceset="RES-US" device="1206"/>
-<part name="R9" library="fab" deviceset="RES-US" device="1206"/>
-<part name="R14" library="fab" deviceset="RES-US" device="1206FAB"/>
-<part name="R16" library="fab" deviceset="RES-US" device="1206FAB"/>
-<part name="C1" library="fab" deviceset="CAP-US" device="1206FAB"/>
+<part name="R2" library="fab" deviceset="RES-US" device="1206FAB" value="0"/>
+<part name="R3" library="fab" deviceset="RES-US" device="1206FAB" value="0"/>
+<part name="R4" library="fab" deviceset="RES-US" device="1206FAB" value="0"/>
+<part name="R10" library="fab" deviceset="RES-US" device="1206FAB" value="0"/>
+<part name="R11" library="fab" deviceset="RES-US" device="1206FAB" value="0"/>
+<part name="R12" library="fab" deviceset="RES-US" device="1206" value="0"/>
+<part name="R13" library="fab" deviceset="RES-US" device="1206" value="0"/>
+<part name="R15" library="fab" deviceset="RES-US" device="1206FAB" value="0"/>
+<part name="R5" library="fab" deviceset="RES-US" device="1206FAB" value="0"/>
+<part name="R6" library="fab" deviceset="RES-US" device="1206" value="0"/>
+<part name="R7" library="fab" deviceset="RES-US" device="1206" value="0"/>
+<part name="R8" library="fab" deviceset="RES-US" device="1206" value="0"/>
+<part name="R9" library="fab" deviceset="RES-US" device="1206" value="0"/>
+<part name="R14" library="fab" deviceset="RES-US" device="1206FAB" value="0"/>
+<part name="R16" library="fab" deviceset="RES-US" device="1206FAB" value="0"/>
+<part name="C1" library="fab" deviceset="CAP-US" device="1206FAB" value=".1uF"/>
 </parts>
 <sheets>
