File: Hardware/MotorControlBoard/motorcontrol.sch (EAGLE design)
At the start: 27 parts, among them U1 ATMEGA328P-AU

Commit message: new board
Parts:
- removed R5: 0, fab:RES-US1206FAB
- removed R6, R7, R8, R9: 0, fab:RES-US1206
Connections:
- removed net N$1: R5.1, U$3.VSS
- removed net N$2: R6.1, U$3.B
- removed net N$3: R7.1, U$3.DGND
- removed net N$4: R8.1, U$3.A
- removed net N$5: R9.2, U$3.CS
- net IN1A: now also U$3.B; no longer R6.2
- net IN1B: now also U$3.DGND; no longer R7.2
- net IN2A: now also U$3.A; no longer R8.2
- net IN2B: now also U$3.CS; no longer R9.1
- net VCC: now also U$3.VSS; no longer R5.2
Changed lines of the file:
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@@
 <part name="R13" library="fab" deviceset="RES-US" device="1206" value="0"/>
 <part name="R15" library="fab" deviceset="RES-US" device="1206FAB" value="0"/>
-<part name="R5" library="fab" deviceset="RES-US" device="1206FAB" value="0"/>
-<part name="R6" library="fab" deviceset="RES-US" device="1206" value="0"/>
-<part name="R7" library="fab" deviceset="RES-US" device="1206" value="0"/>
-<part name="R8" library="fab" deviceset="RES-US" device="1206" value="0"/>
-<part name="R9" library="fab" deviceset="RES-US" device="1206" value="0"/>
 <part name="R14" library="fab" deviceset="RES-US" device="1206FAB" value="0"/>
 <part name="R16" library="fab" deviceset="RES-US" device="1206FAB" value="0"/>
@@
 <instance part="R13" gate="G$1" x="30.48" y="12.7"/>
 <instance part="R15" gate="G$1" x="101.6" y="60.96"/>
-<instance part="R5" gate="G$1" x="144.78" y="96.52"/>
-<instance part="R6" gate="G$1" x="144.78" y="101.6"/>
-<instance part="R7" gate="G$1" x="129.54" y="88.9"/>
-<instance part="R8" gate="G$1" x="144.78" y="111.76"/>
-<instance part="R9" gate="G$1" x="91.44" y="99.06"/>
 <instance part="R14" gate="G$1" x="12.7" y="25.4"/>
 <instance part="R16" gate="G$1" x="142.24" y="66.04"/>
@@
 </segment>
 <segment>
-<pinref part="R5" gate="G$1" pin="2"/>
-<wire x1="149.86" y1="96.52" x2="154.94" y2="96.52" width="0.1524" layer="91"/>
 <label x="154.94" y="96.52" size="1.778" layer="95"/>
+<pinref part="U$3" gate="G$1" pin="VSS"/>
+<wire x1="139.7" y1="96.52" x2="154.94" y2="96.52" width="0.1524" layer="91"/>
 </segment>
 <segment>
@@
 </segment>
 <segment>
-<pinref part="R9" gate="G$1" pin="1"/>
-<wire x1="86.36" y1="99.06" x2="78.74" y2="99.06" width="0.1524" layer="91"/>
 <label x="78.74" y="99.06" size="1.778" layer="95"/>
+<pinref part="U$3" gate="G$1" pin="CS"/>
+<wire x1="96.52" y1="99.06" x2="78.74" y2="99.06" width="0.1524" layer="91"/>
 </segment>
 </net>
@@
 </segment>
 <segment>
-<pinref part="R8" gate="G$1" pin="2"/>
-<wire x1="149.86" y1="111.76" x2="157.48" y2="111.76" width="0.1524" layer="91"/>
 <label x="152.4" y="111.76" size="1.778" layer="95"/>
+<pinref part="U$3" gate="G$1" pin="A"/>
+<wire x1="157.48" y1="111.76" x2="139.7" y2="111.76" width="0.1524" layer="91"/>
 </segment>
 </net>
@@
 </segment>
 <segment>
-<pinref part="R6" gate="G$1" pin="2"/>
-<wire x1="149.86" y1="101.6" x2="154.94" y2="101.6" width="0.1524" layer="91"/>
 <label x="152.4" y="101.6" size="1.778" layer="95"/>
+<pinref part="U$3" gate="G$1" pin="B"/>
+<wire x1="154.94" y1="101.6" x2="139.7" y2="101.6" width="0.1524" layer="91"/>
 </segment>
 </net>
@@
 </segment>
 <segment>
-<pinref part="R7" gate="G$1" pin="2"/>
-<wire x1="134.62" y1="88.9" x2="139.7" y2="88.9" width="0.1524" layer="91"/>
 <label x="137.16" y="88.9" size="1.778" layer="95"/>
+<pinref part="U$3" gate="G$1" pin="DGND"/>
+<wire x1="124.46" y1="88.9" x2="139.7" y2="88.9" width="0.1524" layer="91"/>
 </segment>
 </net>
@@
 </segment>
 </net>
-<net name="N$1" class="0">
-<segment>
-<pinref part="U$3" gate="G$1" pin="VSS"/>
-<pinref part="R5" gate="G$1" pin="1"/>
-</segment>
-</net>
-<net name="N$2" class="0">
-<segment>
-<pinref part="U$3" gate="G$1" pin="B"/>
-<pinref part="R6" gate="G$1" pin="1"/>
-</segment>
-</net>
-<net name="N$3" class="0">
-<segment>
-<pinref part="U$3" gate="G$1" pin="DGND"/>
-<pinref part="R7" gate="G$1" pin="1"/>
-</segment>
-</net>
-<net name="N$4" class="0">
-<segment>
-<pinref part="U$3" gate="G$1" pin="A"/>
-<pinref part="R8" gate="G$1" pin="1"/>
-</segment>
-</net>
-<net name="N$5" class="0">
-<segment>
-<pinref part="U$3" gate="G$1" pin="CS"/>
-<pinref part="R9" gate="G$1" pin="2"/>
-</segment>
-</net>
