File: Hardware/MotorControlBoard/motorcontrol.brd (EAGLE design)
At the start: 52.5 x 39 mm, 27 parts, among them U1 ATMEGA328P-AU

Commit message: changes in eagle file
Parts:
- 1UF: value CAP-US1206FAB -> 1uF
- C1, C2: value CAP-US1206FAB -> .1uF
- C3: value CAP-US1206FAB -> 10uF
- R10, R11, R12, R13, R14, R15, R16, R2, R3, R4, R5, R6, R7, R8, R9: value (none) -> 0
Changed lines of the file:
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@@
 <layer number="18" name="Vias" color="2" fill="1" visible="no" active="yes"/>
 <layer number="19" name="Unrouted" color="6" fill="1" visible="no" active="yes"/>
-<layer number="20" name="Dimension" color="15" fill="1" visible="no" active="yes"/>
-<layer number="21" name="tPlace" color="7" fill="1" visible="no" active="yes"/>
-<layer number="22" name="bPlace" color="7" fill="1" visible="no" active="yes"/>
+<layer number="20" name="Dimension" color="15" fill="1" visible="yes" active="yes"/>
+<layer number="21" name="tPlace" color="7" fill="1" visible="yes" active="yes"/>
+<layer number="22" name="bPlace" color="7" fill="1" visible="yes" active="yes"/>
 <layer number="23" name="tOrigins" color="15" fill="1" visible="no" active="yes"/>
 <layer number="24" name="bOrigins" color="15" fill="1" visible="no" active="yes"/>
 <layer number="25" name="tNames" color="15" fill="1" visible="no" active="yes"/>
 <layer number="26" name="bNames" color="7" fill="1" visible="no" active="yes"/>
-<layer number="27" name="tValues" color="15" fill="1" visible="no" active="yes"/>
-<layer number="28" name="bValues" color="7" fill="1" visible="no" active="yes"/>
+<layer number="27" name="tValues" color="15" fill="1" visible="yes" active="yes"/>
+<layer number="28" name="bValues" color="7" fill="1" visible="yes" active="yes"/>
 <layer number="29" name="tStop" color="7" fill="3" visible="no" active="yes"/>
 <layer number="30" name="bStop" color="7" fill="6" visible="no" active="yes"/>
-<layer number="31" name="tCream" color="7" fill="4" visible="no" active="yes"/>
-<layer number="32" name="bCream" color="7" fill="5" visible="no" active="yes"/>
+<layer number="31" name="tCream" color="7" fill="4" visible="yes" active="yes"/>
+<layer number="32" name="bCream" color="7" fill="5" visible="yes" active="yes"/>
 <layer number="33" name="tFinish" color="6" fill="3" visible="no" active="yes"/>
 <layer number="34" name="bFinish" color="6" fill="6" visible="no" active="yes"/>
 <layer number="35" name="tGlue" color="7" fill="4" visible="no" active="yes"/>
 <layer number="36" name="bGlue" color="7" fill="5" visible="no" active="yes"/>
-<layer number="37" name="tTest" color="7" fill="1" visible="no" active="yes"/>
-<layer number="38" name="bTest" color="7" fill="1" visible="no" active="yes"/>
+<layer number="37" name="tTest" color="7" fill="1" visible="yes" active="yes"/>
+<layer number="38" name="bTest" color="7" fill="1" visible="yes" active="yes"/>
 <layer number="39" name="tKeepout" color="4" fill="11" visible="no" active="yes"/>
 <layer number="40" name="bKeepout" color="1" fill="11" visible="no" active="yes"/>
@@
 <layer number="47" name="Measures" color="7" fill="1" visible="no" active="yes"/>
 <layer number="48" name="Document" color="7" fill="1" visible="no" active="yes"/>
-<layer number="49" name="Reference" color="7" fill="1" visible="no" active="yes"/>
+<layer number="49" name="Reference" color="7" fill="1" visible="yes" active="yes"/>
 <layer number="50" name="dxf" color="7" fill="1" visible="no" active="no"/>
 <layer number="51" name="tDocu" color="7" fill="1" visible="no" active="yes"/>
@@
 <layer number="99" name="SpiceOrder" color="5" fill="1" visible="no" active="no"/>
 <layer number="100" name="Muster" color="7" fill="1" visible="no" active="no"/>
-<layer number="101" name="Patch_Top" color="12" fill="4" visible="no" active="yes"/>
+<layer number="101" name="Patch_Top" color="12" fill="4" visible="yes" active="yes"/>
 <layer number="102" name="Vscore" color="7" fill="1" visible="no" active="yes"/>
 <layer number="103" name="tMap" color="7" fill="1" visible="no" active="yes"/>
@@
 <element name="U$2" library="fab" package="EFOBM" value="RESONATOR" x="13.18895" y="11.71575" rot="R270"/>
 <element name="AVR-ISP" library="fab" package="2X03SMD" value="" x="21.57095" y="7.5311" rot="R90"/>
-<element name="1UF" library="fab" package="C1206FAB" value="CAP-US1206FAB" x="19.558" y="31.1912"/>
-<element name="C2" library="fab" package="C1206FAB" value="CAP-US1206FAB" x="38.6588" y="18.1102" rot="R90"/>
-<element name="C3" library="fab" package="C1206FAB" value="CAP-US1206FAB" x="36.1696" y="18.0594" rot="R90"/>
+<element name="1UF" library="fab" package="C1206FAB" value="1uF" x="19.558" y="31.1912"/>
+<element name="C2" library="fab" package="C1206FAB" value=".1uF" x="38.6588" y="18.1102" rot="R90"/>
+<element name="C3" library="fab" package="C1206FAB" value="10uF" x="36.1696" y="18.0594" rot="R90"/>
 <element name="R1" library="fab" package="R1206FAB" value="10K" x="19.5834" y="28.1178"/>
 <element name="U$3" library="BillPorter" package="MSOP_10" value="AD5290" x="37.3126" y="22.987" rot="R90"/>
 <element name="U$4" library="fab" package="2X02SMD" value="PINHD-2X2-SMD" x="31.1912" y="27.5844" rot="R180"/>
 <element name="0OHM" library="fab" package="R1206FAB" value="" x="37.592" y="12.827" rot="R270"/>
-<element name="R2" library="fab" package="R1206FAB" value="" x="32.512" y="19.558"/>
-<element name="R3" library="fab" package="R1206FAB" value="" x="30.099" y="16.002"/>
-<element name="R4" library="fab" package="R1206FAB" value="" x="19.939" y="34.798" rot="R90"/>
-<element name="R10" library="fab" package="R1206FAB" value="" x="12.319" y="19.304" rot="R90"/>
-<element name="R11" library="fab" package="R1206FAB" value="" x="8.001" y="17.399"/>
-<element name="R12" library="fab" package="R1206" value="" x="32.385" y="9.652" rot="R180"/>
-<element name="R13" library="fab" package="R1206" value="" x="27.559" y="10.414" rot="R180"/>
-<element name="R15" library="fab" package="R1206FAB" value="" x="23.368" y="34.798" rot="R90"/>
-<element name="R5" library="fab" package="R1206FAB" value="" x="46.99" y="21.209" rot="R270"/>
-<element name="R6" library="fab" package="R1206" value="" x="44.704" y="15.621" rot="R270"/>
-<element name="R7" library="fab" package="R1206" value="" x="45.466" y="27.051" rot="R90"/>
-<element name="R8" library="fab" package="R1206" value="" x="41.91" y="19.431" rot="R270"/>
-<element name="R9" library="fab" package="R1206" value="" x="42.164" y="26.416" rot="R270"/>
-<element name="R14" library="fab" package="R1206FAB" value="" x="28.702" y="3.937" rot="R90"/>
-<element name="R16" library="fab" package="R1206FAB" value="" x="7.112" y="22.606" rot="R180"/>
-<element name="C1" library="fab" package="C1206FAB" value="CAP-US1206FAB" x="14.732" y="28.575" rot="R90"/>
+<element name="R2" library="fab" package="R1206FAB" value="0" x="32.512" y="19.558"/>
+<element name="R3" library="fab" package="R1206FAB" value="0" x="30.099" y="16.002"/>
+<element name="R4" library="fab" package="R1206FAB" value="0" x="19.939" y="34.798" rot="R90"/>
+<element name="R10" library="fab" package="R1206FAB" value="0" x="12.319" y="19.304" rot="R90"/>
+<element name="R11" library="fab" package="R1206FAB" value="0" x="8.001" y="17.399"/>
+<element name="R12" library="fab" package="R1206" value="0" x="32.385" y="9.652" rot="R180"/>
+<element name="R13" library="fab" package="R1206" value="0" x="27.559" y="10.414" rot="R180"/>
+<element name="R15" library="fab" package="R1206FAB" value="0" x="23.368" y="34.798" rot="R90"/>
+<element name="R5" library="fab" package="R1206FAB" value="0" x="46.99" y="21.209" rot="R270"/>
+<element name="R6" library="fab" package="R1206" value="0" x="44.704" y="15.621" rot="R270"/>
+<element name="R7" library="fab" package="R1206" value="0" x="45.466" y="27.051" rot="R90"/>
+<element name="R8" library="fab" package="R1206" value="0" x="41.91" y="19.431" rot="R270"/>
+<element name="R9" library="fab" package="R1206" value="0" x="42.164" y="26.416" rot="R270"/>
+<element name="R14" library="fab" package="R1206FAB" value="0" x="28.702" y="3.937" rot="R90"/>
+<element name="R16" library="fab" package="R1206FAB" value="0" x="7.112" y="22.606" rot="R180"/>
+<element name="C1" library="fab" package="C1206FAB" value=".1uF" x="14.732" y="28.575" rot="R90"/>
 </elements>
 <signals>

Commit message: new case
Parts:
- removed R5: 0, fab:R1206FAB
- removed R6, R7, R8, R9: 0, fab:R1206
Connections:
- removed net N$1: R5.1, U$3.3
- removed net N$2: R6.1, U$3.2
- removed net N$3: R7.1, U$3.4
- removed net N$4: R8.1, U$3.1
- removed net N$5: R9.2, U$3.5
- net IN1A: now also U$3.2; no longer R6.2
- net IN1B: now also U$3.4; no longer R7.2
- net IN2A: now also U$3.1; no longer R8.2
- net IN2B: now also U$3.5; no longer R9.1
- net RX: now also U$1.4; no longer U$1.5
- net TX: now also U$1.5; no longer U$1.4
- net VCC: now also U$3.3; no longer R5.2
Routing:
- net N$9: track 183.1 -> 0.00 mm
- net VCC: track 148.3 -> 49.5 mm
- net GND: track 76.5 -> 35.2 mm
- net TX: track 18.7 -> 0.00 mm
- net RX: track 16.7 -> 0.00 mm
- net N$2: track 10.7 -> 0.00 mm
- net N$7: track 10.2 -> 0.00 mm
- net N$3: track 8.24 -> 0.00 mm
- net N$1: track 7.69 -> 0.00 mm
- net N$5: track 3.75 -> 0.00 mm
- net N$4: track 3.62 -> 0.00 mm
- net IN1B: track 36.4 -> 32.9 mm
- net N$10: track 2.21 -> 0.00 mm
- net IN1A: track 25.7 -> 24.3 mm
