File: Hardware/MotorControlBoard/motorcontrol_v2.brd (EAGLE design)
At the start: 52.5 x 39 mm, 27 parts, among them U1 ATMEGA328P-AU

Commit message: new case
Parts:
- removed R9: 0, fab:R1206
- R5: value 0 -> (none)
- R6: value 0 -> (none); device fab:R1206 -> fab:R1206FAB
- R7, R8: device fab:R1206 -> fab:R1206FAB
- moved R5 37.8 mm to (14.4, 40.3), turned to 180 degrees
- moved R3 31.4 mm to (30.5, 47.4), turned to 270 degrees
- moved R6 26.1 mm to (27.2, 34.9), turned to 90 degrees
- moved R7 25.9 mm to (25.0, 11.2), turned to 270 degrees
- moved R16 24.0 mm to (19.7, 43.1), turned to 90 degrees
- moved R4 17.7 mm to (33.7, 46.0)
- moved R15 17.2 mm to (36.4, 46.0)
- moved R10 17.0 mm to (26.5, 28.7)
- moved U$2 17.0 mm to (28.2, 19.8)
- moved U1 16.5 mm to (34.0, 28.3)
- moved C1 16.5 mm to (25.4, 41.1)
- moved R1 16.5 mm to (32.0, 38.9)
- moved 1UF 16.4 mm to (32.0, 41.9)
- moved R11 16.3 mm to (24.3, 16.4)
- moved R2 15.3 mm to (44.6, 28.9), turned to 45 degrees
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Connections:
- removed net N$11: R2.1, R3.2
- removed net N$5: R9.2, U$3.5
- new net GNDDD: R2.1, R8.1, U1.21
- net CTS: now also R6.1; no longer R16.1
- net GNDD: now also R8.2; no longer R3.1, U1.21
- net IN1A: now also U$3.2; no longer R6.2
- net IN1B: now also U$3.4; no longer R7.2
- net IN2A: now also U$3.1; no longer R8.2
- net IN2B: now also U$3.5; no longer R9.1
- net N$1: now also R5.2, U$1.4; no longer R5.1, U$3.3
- net N$2: now also R16.1, R6.2; no longer R6.1, U$3.2
- net N$3: now also 1UF.1, R1.1, R3.2; no longer R7.1, U$3.4
- net N$4: now also R3.1, R7.2; no longer R8.1, U$3.1
- net RX: now also R5.1; no longer U$1.4
- net VCC: now also R7.1, U$3.3; no longer 1UF.1, R1.1, R5.2
Routing:
- net N$9: track 183.1 -> 0.00 mm
- net N$4: track 3.62 -> 77.7 mm
- net VCC: track 148.3 -> 75.5 mm
- net N$7: track 10.2 -> 40.1 mm
- net GND: track 76.5 -> 104.3 mm
- net N$10: track 2.21 -> 26.9 mm
- net JUMP2: track 32.2 -> 13.2 mm
- net N$1: track 7.69 -> 20.3 mm
- net GNDD: track 23.6 -> 12.0 mm
- net MOSI: track 4.28 -> 14.7 mm
- net RST: track 17.9 -> 28.1 mm
- net JUMP: track 82.6 -> 72.9 mm
- net RX: track 16.5 -> 25.8 mm
- net GNDDD: track 0.00 -> 7.27 mm
- net IN1B: track 36.4 -> 30.9 mm
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
Commit message: new board stuff
Parts:
- removed U$2: RESONATOR, fab:EFOBM
- added 20MHZ: 20MHZ, fab:EFOBM
- 0OHM, R5, R6: value (none) -> 0
- moved 0OHM 6.37 mm to (40.3, 25.0)
- moved C2 6.37 mm to (42.6, 28.4)
- moved C3 6.37 mm to (40.7, 28.3)
- moved R1 6.37 mm to (25.7, 39.4)
- moved R11 6.37 mm to (17.9, 16.9)
- moved R12 6.37 mm to (33.8, 18.3)
- moved R14 6.37 mm to (35.3, 12.4)
- moved R3 6.37 mm to (24.1, 47.9)
- moved R4 6.37 mm to (27.3, 46.5)
- moved R5 6.37 mm to (8.00, 40.8)
- moved R6 6.37 mm to (20.8, 35.4)
- moved R8 6.37 mm to (35.7, 26.0)
- moved U$4 6.37 mm to (35.9, 38.0)
- moved U$1 6.37 mm to (15.7, 28.6)
- moved 1UF 6.37 mm to (25.7, 42.4)
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Connections:
- net GNA: now also 20MHZ.2; no longer U$2.2
- net R1: now also 20MHZ.1; no longer U$2.1
- net R2: now also 20MHZ.3; no longer U$2.3
Other:
- board size 52.5 x 39 mm -> 50.8 x 76.2 mm
- board text added: "Open S Pump V0.1"

Commit message: lots of changes
Parts:
- removed 20MHZ: 20MHZ, fab:EFOBM
- added U$2: RESONATOR, fab:EFOBM
- 0OHM, R5, R6: value 0 -> (none)
- moved 0OHM 6.37 mm to (46.6, 24.5)
- moved C2 6.37 mm to (48.9, 27.9)
- moved C3 6.37 mm to (47.1, 27.8)
- moved R1 6.37 mm to (32.0, 38.9)
- moved R11 6.37 mm to (24.3, 16.4)
- moved R12 6.37 mm to (40.1, 17.8)
- moved R14 6.37 mm to (41.7, 11.9)
- moved R3 6.37 mm to (30.5, 47.4)
- moved R4 6.37 mm to (33.7, 46.0)
- moved R5 6.37 mm to (14.4, 40.3)
- moved R6 6.37 mm to (27.2, 34.9)
- moved R8 6.37 mm to (42.0, 25.5)
- moved U$4 6.37 mm to (42.2, 37.5)
- moved U$1 6.37 mm to (22.1, 28.1)
- moved 1UF 6.37 mm to (32.0, 41.9)
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Connections:
- net GNA: now also U$2.2; no longer 20MHZ.2
- net R1: now also U$2.1; no longer 20MHZ.1
- net R2: now also U$2.3; no longer 20MHZ.3
Other:
- board size 50.8 x 76.2 mm -> 52.5 x 39 mm
- board text removed: "Open S Pump V0.1"
